File: extras/SoftstartPlugIn.sch (EAGLE design)
At the start: 27 parts, among them U1 ATTINY85

Commit message: Documentation
Parts:
- removed CX3: 100n, rcl:CXXC15B5
- removed INT_BREMSWICKLUNG: (no value), rcl:L-EUIR-2
- removed S1: (no value), e-schalter:DRUCK-WECHSELSCHALTER
- added D8, D9: BAT42, diode:BAT42
- added L1: 82114A, inductors:82114A
- added R10, R8: 6.8M, rcl:R-EU_0207/10
- CX2: value 100n -> 200n
- R13: value 1 -> 2.2
Connections:
- removed net N$12: BTA12/600SW.A2, CX1.2, CX3.1, INT_BREMSWICKLUNG.1, MOTOR.X2
- new net N$19: BTA12/600SW.A2, CX1.2, R8.1
- net +5V: now also D9.C
- net N$15: now also MOTOR.X2; no longer S1.14
- net N$16: now also R10.1, R8.2; no longer INT_BREMSWICKLUNG.2, S1.12
- net N$17: now also D8.A, D8.C, D9.A, R10.2, U1.PB1
- net N$18: now also MOTOR.X1; no longer U1.PB1
- net N$8: no longer CX3.2, MOTOR.X1, S1.11
Other:
- note added: "Capacitive power supply"
- note added: "Load detection"
- note added: "X2 for 230 volt AC"
- moved on the sheet: MOTOR
